File: AudioBoard4.sch (EAGLE design)
At the start: 294 parts, among them IC1 TL084D, IC10 TL084D, IC11 TL074D, IC13 SSM2164P, IC14 TL071D, IC15 TL084D, IC16 TL071D, IC17 TL084D, IC18 SSM2164P, IC19 TL071D, IC2 TL074D, IC20 TL084D, IC21 TL071D, IC22 TL084D, IC23 TL072D, IC24 LT1054, IC25 7905, IC26 7805, IC4 TL084D, IC5 TL074D, IC7 TL084D, IC8 TL074D

Commit message: Update eagle files to contain powerdown signal.
Parts:
- removed C100, C101, C102, C103, C104, C105, C106, C107, C108, C111, C112, C75, C76, C77, C78, C79, C80, C81, C82, C83, C84, C99: 100n, SparkFun-Capacitors:CAP0603-CAP
- removed C109: 100p, SparkFun-Capacitors:CAP_POL1206
- removed C11, C26, C41, C56: 100pF, SparkFun-Capacitors:CAP0603-CAP
- removed C110: 18p, SparkFun-Capacitors:CAP_POL1206
- removed C113: 100u, rcl:CPOL-USE2.5-6
- removed C114, C115: 220u, rcl:CPOL-USE5-10.5
- removed C116, C117: 100u, rcl:CPOL-USE2.5-7
- removed C118: 10p, rcl:C-US025-025X050
- removed C119: 10u, rcl:CPOL-USE2.5-5
- removed C12, C13, C14, C15, C24, C25, C27, C28, C29, C30, C39, C40, C42, C43, C44, C45, C54, C55, C57, C58, C59, C60: 100nF, SparkFun-Capacitors:CAP0603-CAP
- removed C120, C121: 100n, rcl:C-US025-025X050
- removed C16, C17, C31, C32, C46, C47: 22nF, SparkFun-Capacitors:CAP0603-CAP
- removed C18, C33, C48: (no value), SparkFun-Capacitors:CAP_POL1206-KIT
- removed C19, C34, C49: 1.5nF, SparkFun-Capacitors:CAP0603-CAP
- removed C20, C21, C22, C35, C36, C37, C50, C51, C52: 10n, SparkFun-Passives:CAP_POLPTH1
- removed C23, C38, C53: 820p, SparkFun-Capacitors:CAP_POLPTH1
- removed C61, C68, C85, C92: 1uF, SparkFun-Capacitors:100UF-25V-20%(PTH)
- removed C62, C67, C69, C74, C86, C91, C93, C98: 560p, SparkFun-Capacitors:CAP0603-CAP
- removed C63, C66, C70, C73, C87, C90, C94, C97: 100p, SparkFun-Capacitors:CAP0603-CAP
- removed C64, C71, C88, C95: 10uF, SparkFun-Capacitors:100UF-25V-20%(PTH)
- removed C65, C72, C89, C96: 33nF, SparkFun-Capacitors:CAP0603-CAP
- removed D1: 1N4001, diode:1N4004
- removed IC1, IC10, IC15, IC17, IC20, IC22, IC4, IC7: TL084D, linear:TL084D
- removed IC11, IC2, IC5, IC8: TL074D, linear:TL074D
- removed IC12, IC3, IC6, IC9: (no value), ic-package:DIL16
- removed IC13, IC18: SSM2164P, ssm2164:SSM2164P
- removed IC14, IC16, IC19, IC21: TL071D, linear:TL071D
- removed IC23: TL072D, linear:TL072D
- removed IC24: LT1054, ic-package:DIL8
- removed IC25: 7905, v-reg:79XXS
- removed IC26: 7805, v-reg:78XXS
- removed J1: (no value), con-jack2:JACK-PLUG2
- removed JP1, JP2, JP3, JP4, JP5: AUDIO-JACK4-.25-HORIZ-TRS, SparkFun-Connectors:AUDIO-JACK4-.25-HORIZ-TRS
- removed R10, R108, R109, R110, R12, R120, R121, R122, R14, R24, R29, R30, R32, R34, R4, R44, R49, R50, R52, R54, R64, R69, R70, R72, R74, R85, R86, R87, R9, R97, R98, R99: 10k, SparkFun-Passives:RESISTOR0603-RES
- removed R100, R111, R123, R88: 100k, pot:TRIM_EU-RJ9W
- removed R101, R112, R124, R89: 50k, pot:TRIM_EU-RJ9W
- removed R102, R113, R125, R133, R134, R21, R41, R61, R90: 100k, SparkFun-Passives:RESISTOR0603-RES
- removed R103, R105, R114, R117, R126, R135, R136, R137, R138, R139, R82, R91, R94: 470, SparkFun-Passives:RESISTOR0603-RES
- removed R104, R116, R22, R42, R62, R81, R93: 33k, SparkFun-Passives:RESISTOR0603-RES
- removed R106, R118, R20, R40, R60, R80, R83, R95: 47k, SparkFun-Passives:RESISTOR0603-RES
- removed R107, R119, R15, R35, R55, R75, R84, R96: 150, SparkFun-Passives:RESISTOR0603-RES
- removed R11, R23, R28, R3, R31, R43, R48, R51, R63, R68, R71, R8: 22k, SparkFun-Passives:RESISTOR0603-RES
- removed R115, R92: 4.7k, SparkFun-Passives:RESISTOR0603-RES
- removed R127, R128, R129, R130: 10K, SparkFun-Passives:RESISTOR0603-RES
- removed R13, R33, R53, R73: INPUT_LVL, pot:TRIM_EU-RJ9W
- removed R131: RGAIN, SparkFun-Passives:RESISTOR0603-RES
- removed R132: 100K, pot:TRIM_EU-RJ9W
- removed R16, R19, R36, R39, R56, R59, R76, R79: 220, SparkFun-Passives:RESISTOR0603-RES
- removed R17, R37, R57, R77: OFFS_ADJ, pot:TRIM_EU-RJ9W
- removed R18, R38, R58, R78: 390k, SparkFun-Passives:RESISTOR0603-RES
- removed R25, R45, R5, R65: 1k, SparkFun-Passives:RESISTOR0603-RES
- removed R26, R46, R6, R66: 68k, SparkFun-Passives:RESISTOR0603-RES
- removed R27, R47, R67, R7: 330k, SparkFun-Passives:RESISTOR0603-RES
- removed SW: (no value), SparkFun:M02PTH
- added INA, INB, OUTA, OUTB: (no value), adafruit:PINHD-1X3
- added L1, L2: 10uH, SparkFun-Passives:INDUCTOR0805
- added L3: 10uH, SparkFun-Passives:INDUCTOR0603
- added U$1: TEENSY_3.0_ALL_PINS_AND_PADS, Teensy_3_Series_Board_v1.0:TEENSY_3.0_ALL_PINS_AND_PADS
- added U$2, U$3: AK4558EN, AK4558:AK4558EN
- C1, C2: value 22nF -> 100n; device SparkFun-Capacitors:CAP0603-CAP -> SparkFun-Passives:CAP0603-CAP
- C10, C9: value 100nF -> 100n; device SparkFun-Capacitors:CAP0603-CAP -> SparkFun-Passives:CAP0603-CAP
- C3: value (none) -> 100n; device SparkFun-Capacitors:CAP_POL1206-KIT -> SparkFun-Passives:CAP0603-CAP
- C4: value 1.5nF -> 100n; device SparkFun-Capacitors:CAP0603-CAP -> SparkFun-Passives:CAP0603-CAP
- C5, C6, C7: value 10n -> 100n; device SparkFun-Passives:CAP_POLPTH1 -> SparkFun-Passives:CAP0603-CAP
- C8: value 820p -> 100n; device SparkFun-Capacitors:CAP_POLPTH1 -> SparkFun-Passives:CAP0603-CAP
- R1: value 100k -> 1k
- R2: value 33k -> 1k
Connections:
- removed net N$100: C63.2, IC13B.OUT, IC14.-IN, R83.1
- removed net N$101: C63.1, IC14.OUT, R83.2, R84.1
- removed net N$102: C64.+, R84.2
- removed net N$103: C65.2, R86.2, R87.1
- removed net N$104: C66.2, IC13A.OUT, IC15A.-IN, R87.2
- removed net N$105: C66.1, IC13A.CTRL, IC15A.OUT, IC15B.+IN
- removed net N$106: IC13A.IN, R90.1, R91.2
- removed net N$107: R88.S, R90.2
- removed net N$108: C67.2, R91.1
- removed net N$109: IC13B.CTRL, IC15B.OUT, R89.A
- removed net N$110: IC15B.-IN, R89.S
- removed net N$111: IC13E.MODE, R92.2
- removed net N$112: C68.-, R93.1
- removed net N$113: IC13C.IN, R93.2, R94.2
- removed net N$114: C69.2, R94.1
- removed net N$115: C70.2, IC13C.OUT, IC16.-IN, R95.1
- removed net N$116: C70.1, IC16.OUT, R95.2, R96.1
- removed net N$117: C71.+, R96.2
- removed net N$118: IC13C.CTRL, IC17B.OUT, R101.A
- removed net N$119: C72.2, R98.2, R99.1
- removed net N$120: C73.2, IC13D.OUT, IC17A.-IN, R99.2
- removed net N$121: C73.1, IC13D.CTRL, IC17A.OUT, IC17B.+IN
- removed net N$122: IC13D.IN, R102.1, R103.2
- removed net N$123: R100.S, R102.2
- removed net N$124: C74.2, R103.1
- removed net N$125: IC17B.-IN, R101.S
- removed net N$126: C85.-, R104.1
- removed net N$127: IC18B.IN, R104.2, R105.2
- removed net N$128: C86.2, R105.1
- removed net N$129: C87.2, IC18B.OUT, IC19.-IN, R106.1
- removed net N$130: C87.1, IC19.OUT, R106.2, R107.1
- removed net N$131: C88.+, R107.2
- removed net N$132: C89.2, R109.2, R110.1
- removed net N$133: C90.2, IC18A.OUT, IC20A.-IN, R110.2
- removed net N$134: C90.1, IC18A.CTRL, IC20A.OUT, IC20B.+IN
- removed net N$135: IC18A.IN, R113.1, R114.2
- removed net N$136: R111.S, R113.2
- removed net N$137: C91.2, R114.1
- removed net N$138: IC18B.CTRL, IC20B.OUT, R112.A
- removed net N$139: IC20B.-IN, R112.S
- removed net N$140: IC18E.MODE, R115.2
- removed net N$141: C92.-, R116.1
- removed net N$142: IC18C.IN, R116.2, R117.2
- removed net N$143: C93.2, R117.1
- removed net N$144: C94.2, IC18C.OUT, IC21.-IN, R118.1
- removed net N$145: C94.1, IC21.OUT, R118.2, R119.1
- removed net N$146: C95.+, R119.2
- removed net N$147: IC18C.CTRL, IC22B.OUT, R124.A
- removed net N$148: C96.2, R121.2, R122.1
- removed net N$149: C97.2, IC18D.OUT, IC22A.-IN, R122.2
- removed net N$150: C97.1, IC18D.CTRL, IC22A.OUT, IC22B.+IN
- removed net N$151: IC18D.IN, R125.1, R126.2
- removed net N$152: R123.S, R125.2
- removed net N$153: C98.2, R126.1
- removed net N$154: IC22B.-IN, R124.S
- removed net N$155: C109.+, IC23B.-IN, R127.2, R128.2, R129.2, R130.2, R131.1
- removed net N$156: C109.-, IC23B.OUT, R131.2, R132.E
- removed net N$157: R132.S, R133.1
- removed net N$158: C110.+, IC23A.-IN, R133.2, R134.1
- removed net N$159: C110.-, JP5.TIP, R134.2, R135.2
- removed net N$160: IC23A.OUT, R135.1
- removed net N$161: JP1.TIP-NORM, R127.1
- removed net N$162: JP2.TIP-NORM, R128.1
- removed net N$163: JP3.TIP-NORM, R129.1
- removed net N$164: JP4.TIP-NORM, R130.1
- removed net N$165: JP1.TIP, R136.1
- removed net N$166: JP2.TIP, R137.1
- removed net N$167: JP3.TIP, R138.1
- removed net N$168: JP4.TIP, R139.1
- removed net N$169: J1.3, SW.1
- removed net N$17: C7.+, IC3.12
- removed net N$170: C116.+, D1.C, IC24.8, IC26.IN
- removed net N$171: C113.+, C118.1, C119.+, IC24.2
- removed net N$172: C113.-, C119.-, IC24.4
- removed net N$173: C117.-, IC24.5, IC25.IN
- removed net N$174: D1.A, SW.2
- removed net N$175: C118.2, IC24.7
- removed net N$18: C5.+, IC3.6
- removed net N$19: C8.+, IC3.4
- removed net N$20: C6.-, IC3.11
- removed net N$21: C7.-, IC3.14
- removed net N$22: C16.1, IC4D.-IN, R21.2, R22.2, R23.1
- removed net N$23: R17.S, R18.2
- removed net N$24: IC3.15, R18.1, R19.2
- removed net N$25: C11.1, IC2D.-IN, IC3.3, R20.1
- removed net N$26: C16.2, IC4D.OUT, R23.2, R24.1
- removed net N$27: IC6.13, R24.2, R25.2
- removed net N$28: C17.1, IC4A.-IN, R26.2, R27.2, R28.1
- removed net N$29: C17.2, IC4A.OUT, R28.2, R29.1
- removed net N$3: IC3.13, R4.2, R5.2
- removed net N$30: IC4B.-IN, R29.2, R30.1
- removed net N$31: IC4B.OUT, R30.2, R35.1
- removed net N$32: C19.1, IC5C.-IN, R31.1, R32.2
- removed net N$33: C18.-, R31.2
- removed net N$34: C19.2, IC5C.OUT, R32.1, R33.A
- removed net N$35: R33.E, R33.S, R34.1
- removed net N$36: IC6.2, R35.2
- removed net N$37: IC6.1, R34.2, R36.1
- removed net N$38: C20.-, IC6.7
- removed net N$39: C23.-, IC6.5
- removed net N$40: C21.+, IC6.10
- removed net N$41: C22.+, IC6.12
- removed net N$42: C20.+, IC6.6
- removed net N$43: C23.+, IC6.4
- removed net N$44: C21.-, IC6.11
- removed net N$45: C22.-, IC6.14
- removed net N$46: R37.S, R38.2
- removed net N$47: IC6.15, R38.1, R39.2
- removed net N$48: C26.1, IC5D.-IN, IC6.3, R40.1
- removed net N$49: C31.1, IC7D.-IN, R41.2, R42.2, R43.1
- removed net N$5: C2.2, IC1A.OUT, R8.2, R9.1
- removed net N$50: C31.2, IC7D.OUT, R43.2, R44.1
- removed net N$51: IC9.13, R44.2, R45.2
- removed net N$52: C32.1, IC7A.-IN, R46.2, R47.2, R48.1
- removed net N$53: C32.2, IC7A.OUT, R48.2, R49.1
- removed net N$54: IC7B.-IN, R49.2, R50.1
- removed net N$55: IC7B.OUT, R50.2, R55.1
- removed net N$56: C34.1, IC8C.-IN, R51.1, R52.2
- removed net N$57: C33.-, R51.2
- removed net N$58: C34.2, IC8C.OUT, R52.1, R53.A
- removed net N$59: R53.E, R53.S, R54.1
- removed net N$60: IC9.2, R55.2
- removed net N$61: IC9.1, R54.2, R56.1
- removed net N$62: C35.-, IC9.7
- removed net N$63: C38.-, IC9.5
- removed net N$64: C36.+, IC9.10
- removed net N$65: C37.+, IC9.12
- removed net N$66: C35.+, IC9.6
- removed net N$67: C38.+, IC9.4
- removed net N$68: C36.-, IC9.11
- removed net N$69: C37.-, IC9.14
- removed net N$70: R57.S, R58.2
- removed net N$71: IC9.15, R58.1, R59.2
- removed net N$72: C41.1, IC8D.-IN, IC9.3, R60.1
- removed net N$73: C46.1, IC10D.-IN, R61.2, R62.2, R63.1
- removed net N$74: C46.2, IC10D.OUT, R63.2, R64.1
- removed net N$75: IC12.13, R64.2, R65.2
- removed net N$76: C47.1, IC10A.-IN, R66.2, R67.2, R68.1
- removed net N$77: C47.2, IC10A.OUT, R68.2, R69.1
- removed net N$78: IC10B.-IN, R69.2, R70.1
- removed net N$79: IC10B.OUT, R70.2, R75.1
- removed net N$80: C49.1, IC11C.-IN, R71.1, R72.2
- removed net N$81: C48.-, R71.2
- removed net N$82: C49.2, IC11C.OUT, R72.1, R73.A
- removed net N$83: R73.E, R73.S, R74.1
- removed net N$84: IC12.2, R75.2
- removed net N$85: IC12.1, R74.2, R76.1
- removed net N$86: C50.-, IC12.7
- removed net N$87: C53.-, IC12.5
- removed net N$88: C51.+, IC12.10
- removed net N$89: C52.+, IC12.12
- removed net N$90: C50.+, IC12.6
- removed net N$91: C53.+, IC12.4
- removed net N$92: C51.-, IC12.11
- removed net N$93: C52.-, IC12.14
- removed net N$94: R77.S, R78.2
- removed net N$95: IC12.15, R78.1, R79.2
- removed net N$96: C56.1, IC11D.-IN, IC12.3, R80.1
- removed net N$97: C61.-, R81.1
- removed net N$98: IC13B.IN, R81.2, R82.2
- removed net N$99: C62.2, R82.1
- removed net VCAA_AMP_IN1: R109.1, R86.1
- removed net VCAA_OUT1: C64.-, C88.-, R108.2, R85.2
- removed net VCAA_OUT2: R136.2
- removed net VCAA_OUT3: R138.2
- removed net VCAB_AMP_IN1: R121.1, R98.1
- removed net VCAB_OUT1: C71.-, C95.-, R120.2, R97.2
- removed net VCAB_OUT2: R137.2
- removed net VCAB_OUT3: R139.2
- removed net VCC: C10.2, C102.1, C103.1, C104.1, C106.1, C108.1, C111.1, C114.+, C12.2, C120.1, C13.2, C25.2, C27.2, C28.2, C40.2, C42.2, C43.2, C55.2, C57.2, C58.2, C78.1, C79.1, C80.1, C82.1, C84.1, IC10P.V+, IC11P.V+, IC12.16, IC13E.V+, IC14.V+, IC15P.V+, IC16.V+, IC17P.V+, IC18E.V+, IC19.V+, IC1P.V+, IC20P.V+, IC21.V+, IC22P.V+, IC23P.V+, IC26.OUT, IC2P.V+, IC3.16, IC4P.V+, IC5P.V+, IC6.16, IC7P.V+, IC8P.V+, IC9.16, R115.1, R17.A, R27.1, R37.A, R47.1, R57.A, R67.1, R7.1, R77.A, R92.1
- removed net VCF_AUDIO1: C3.+
- removed net VCF_AUDIO2: C18.+
- removed net VCF_AUDIO3: C33.+
- removed net VCF_AUDIO4: C48.+
- removed net VCF_CUTOFF1: R2.1
- removed net VCF_CUTOFF2: R22.1
- removed net VCF_CUTOFF3: R42.1
- removed net VCF_CUTOFF4: R62.1
- removed net VCF_OUT1: C11.2, C61.+, IC2D.OUT, R20.2
- removed net VCF_OUT2: C26.2, C68.+, IC5D.OUT, R40.2
- removed net VCF_OUT3: C41.2, C85.+, IC8D.OUT, R60.2
- removed net VCF_OUT4: C56.2, C92.+, IC11D.OUT, R80.2
- removed net VCF_RES1: R6.1
- removed net VCF_RES2: R26.1
- removed net VCF_RES3: R46.1
- removed net VCF_RES4: R66.1
- removed net VEE: C100.2, C101.1, C105.1, C107.1, C112.1, C115.-, C121.2, C14.1, C15.1, C24.2, C29.1, C30.1, C39.2, C44.1, C45.1, C54.2, C59.1, C60.1, C75.2, C76.2, C77.1, C81.1, C83.1, C9.2, C99.2, IC10P.V-, IC11P.V-, IC12.9, IC13E.V-, IC14.V-, IC15P.V-, IC16.V-, IC17P.V-, IC18E.V-, IC19.V-, IC1P.V-, IC20P.V-, IC21.V-, IC22P.V-, IC23P.V-, IC25.OUT, IC2P.V-, IC3.9, IC4P.V-, IC5P.V-, IC6.9, IC7P.V-, IC8P.V-, IC9.9, R1.1, R100.A, R111.A, R123.A, R17.E, R21.1, R37.E, R41.1, R57.E, R61.1, R77.E, R88.A
- new net BCLK: U$1.9, U$2.BICK, U$3.BICK
- new net GNDA: C3.2, C4.1, C8.2, C9.1, INA.2, INB.2, L3.2, OUTA.2, OUTB.2, U$2.VSS1, U$3.VSS1
- new net LRCLK: U$1.23/A9, U$2.LRCK, U$3.LRCK
- new net MCLK: U$1.11, U$2.MCKI, U$3.MCKI
- new net PDN: U$1.14/A0, U$2.PDN, U$3.PDN
- new net RX: U$1.13, U$2.SDTO
- new net RX1: U$1.30, U$3.SDTO
- new net SCL: R1.1, U$1.19/A5, U$2.SDA, U$3.SDA
- new net SDA: R2.1, U$1.18/A4, U$2.SCL, U$3.SCL
- new net TX: U$1.22/A8, U$2.SDTI
- new net TX1: U$1.15/A1, U$3.SDTI
- new net VDD: C10.1, C2.1, C5.1, C7.1, L1.1, L2.1, R1.2, R2.2, U$1.3.3V, U$2.LDOE, U$2.TVDD, U$3.CAD0, U$3.LDOE, U$3.TVDD
- net GND: now also C1.2, C10.2, C2.2, C5.2, C6.2, C7.2, L3.1, U$1.GND, U$2.CAD0, U$2.CAD1, U$2.CKS0, U$2.CKS1, U$2.CKS2, U$2.CKS3, U$2.LOPS, U$2.PS, U$2.VCOC, U$2.VSS2, U$3.CAD1, U$3.CKS0, U$3.CKS1, U$3.CKS2, U$3.CKS3, U$3.LOPS, U$3.PS, U$3.VCOC, U$3.VSS2; no longer C10.1, C100.1, C101.2, C102.2, C103.2, C104.2, C105.2, C106.2, C107.2, C108.2, C111.2, C112.2, C114.-, C115.+, C116.-, C117.+, C12.1, C120.2, C121.1, C13.1, C14.2, C15.2, C24.1, C25.1, C27.1, C28.1, C29.2, C30.2, C39.1, C40.1, C42.1, C43.1, C44.2, C45.2, C54.1, C55.1, C57.1, C58.1, C59.2, C60.2, C62.1, C65.1, C67.1, C69.1, C72.1, C74.1, C75.1, C76.1, C77.2, C78.2, C79.2, C80.2, C81.2, C82.2, C83.2, C84.2, C86.1, C89.1, C9.1, C91.1, C93.1, C96.1, C98.1, C99.1, IC10A.+IN, IC10B.+IN, IC10D.+IN, IC11C.+IN, IC11D.+IN, IC12.8, IC13E.GND, IC14.+IN, IC16.+IN, IC18E.GND, IC19.+IN, IC1A.+IN, IC1B.+IN, IC1D.+IN, IC21.+IN, IC23A.+IN, IC23B.+IN, IC24.3, IC25.GND, IC26.GND, IC2C.+IN, IC2D.+IN, IC3.8, IC4A.+IN, IC4B.+IN, IC4D.+IN, IC5C.+IN, IC5D.+IN, IC6.8, IC7A.+IN, IC7B.+IN, IC7D.+IN, IC8C.+IN, IC8D.+IN, IC9.8, J1.1, JP1.EARTH, JP1.EARTH-NORM, JP2.EARTH, JP2.EARTH-NORM, JP3.EARTH, JP3.EARTH-NORM, JP4.EARTH, JP4.EARTH-NORM, JP5.EARTH, JP5.EARTH-NORM, R100.E, R101.E, R108.1, R111.E, R112.E, R120.1, R123.E, R124.E, R132.A, R16.2, R19.1, R25.1, R36.2, R39.1, R45.1, R5.1, R56.2, R59.1, R65.1, R76.2, R79.1, R85.1, R88.E, R89.E, R97.1
- net N$1: now also U$2.VDD18; no longer IC1D.-IN, R1.2, R2.2, R3.1
- net N$10: now also C6.1, U$3.VDD18; no longer C4.2, IC2C.OUT, R12.1, R13.A
- net N$11: now also C8.1, L2.2, U$3.AVDD; no longer R13.E, R13.S, R14.1
- net N$12: now also C9.2, U$3.VCOM; no longer IC3.2, R15.2
- net N$13: now also INB.1, U$3.LIN; no longer IC3.1, R14.2, R16.1
- net N$14: now also INB.3, U$3.RIN; no longer C5.-, IC3.7
- net N$15: now also OUTB.1, U$3.LOUT; no longer C8.-, IC3.5
- net N$16: now also OUTB.3, U$3.ROUT; no longer C6.+, IC3.10
- net N$2: now also C3.1, L1.2, U$2.AVDD; no longer C1.2, IC1D.OUT, R3.2, R4.1
- net N$4: now also C4.2, U$2.VCOM; no longer C2.1, IC1A.-IN, R6.2, R7.2, R8.1
- net N$6: now also INA.1, U$2.LIN; no longer IC1B.-IN, R10.1, R9.2
- net N$7: now also INA.3, U$2.RIN; no longer IC1B.OUT, R10.2, R15.1
- net N$8: now also OUTA.1, U$2.LOUT; no longer C4.1, IC2C.-IN, R11.1, R12.2
- net N$9: now also OUTA.3, U$2.ROUT; no longer C3.-, R11.2
Other:
- note removed: "+/- 5V supply"
- note removed: "<- +/- 90mV"
